Commit message: rename robots

File: precise_description/robots/PF400_long.urdf.xacro (robot description, xacro)
@@ -1,6 +1,6 @@
 <?xml version="1.0"?>
 <robot xmlns:xacro="http://www.ros.org/wiki/xacro"
-       name="PF400">
-  <xacro:property name="yaml_file" value="$(find precise_description)/robots/PF400.yaml"/>
+       name="PF400_long">
+  <xacro:property name="yaml_file" value="$(find precise_description)/robots/PF400_long.yaml"/>
   <xacro:property name="robot_properties" value="${load_yaml(yaml_file)}"/>
   <xacro:include filename="$(find precise_description)/urdf/precise_flex.urdf.xacro"/>

File: precise_description/robots/PF400_short.urdf.xacro (robot description, xacro)
@@ -1,6 +1,6 @@
 <?xml version="1.0"?>
 <robot xmlns:xacro="http://www.ros.org/wiki/xacro"
-       name="PF3400">
-  <xacro:property name="yaml_file" value="$(find precise_description)/robots/PF3400.yaml"/>
+       name="PF400_short">
+  <xacro:property name="yaml_file" value="$(find precise_description)/robots/PF400_short.yaml"/>
   <xacro:property name="robot_properties" value="${load_yaml(yaml_file)}"/>
   <xacro:include filename="$(find precise_description)/urdf/precise_flex.urdf.xacro"/>

Commit message: rename meshes

File: precise_description/robots/PF400_long.urdf.xacro (robot description, xacro)
@@ -5,5 +5,5 @@
   <xacro:property name="robot_properties" value="${load_yaml(yaml_file)}"/>
   <xacro:include filename="$(find precise_description)/urdf/precise_flex.urdf.xacro"/>
-  <xacro:precise_flex name="arm" parent="world">
+  <xacro:precise_flex name="arm" parent="world" has_podest="${True}">
     <origin xyz="0.0 0.0 0.0" rpy="0.0 0.0 0.0"/>
   </xacro:precise_flex>

File: precise_description/robots/PF400_short.urdf.xacro (robot description, xacro)
@@ -5,5 +5,5 @@
   <xacro:property name="robot_properties" value="${load_yaml(yaml_file)}"/>
   <xacro:include filename="$(find precise_description)/urdf/precise_flex.urdf.xacro"/>
-  <xacro:precise_flex name="arm" parent="world">
+  <xacro:precise_flex name="arm" parent="world" has_podest="${True}">
     <origin xyz="0.0 0.0 0.0" rpy="0.0 0.0 0.0"/>
   </xacro:precise_flex>

File: precise_description/urdf/precise_flex.urdf.xacro (robot description, xacro)
@@ -3,5 +3,5 @@
   <xacro:include filename="$(find precise_description)/urdf/materials.xacro"/>
   <xacro:include filename="$(find precise_description)/urdf/transmission.xacro" />
-  <xacro:macro name="precise_flex" params="parent name *origin">
+  <xacro:macro name="precise_flex" params="parent name *origin has_podest:=True">
     <xacro:property name="origin_1_joint">
       <origin xyz="${robot_properties['arm']['arm_1_joint']['origin']['x']} ${robot_properties['arm']['arm_1_joint']['origin']['y']} ${robot_properties['arm']['arm_1_joint']['origin']['z']}" rpy="${robot_properties['arm']['arm_1_joint']['origin']['roll']} ${robot_properties['arm']['arm_1_joint']['origin']['pitch']} ${robot_properties['arm']['arm_1_joint']['origin']['yaw']}"/>
@@ -41,58 +41,82 @@
       <xacro:insert_block name="origin" />
       <parent link="${parent}"/>
-      <child link="z_column" />
-    </joint>
+      <child link="${name}_base_link" />
+    </joint>
+    <link name="${name}_base_link">
+      <xacro:default_inertial/>
+    </link>
+    <joint name="${name}_mount_joint" type="fixed">
+      <origin xyz="0 0 0" rpy="0 0 0"/>
+      <parent link="${name}_base_link"/>
+      <child link="${name}_1_link"/>
+    </joint>
+    <xacro:if value="${has_podest}">
+      <joint name="${name}_podest_joint" type="fixed">
+        <origin xyz="0 0 0" rpy="0 0 0"/>
+        <parent link="${name}_base_link"/>
+        <child link="${name}_podest_link"/>
+      </joint>
+      <link name="${name}_podest_link">
+        <xacro:default_inertial/>
+        <visual>
+          <origin xyz="0 0 0" rpy="0 0 0" />
+          <geometry>
+            <mesh filename="package://precise_description/meshes/arm_podest_link.STL"/>
+          </geometry>
+        </visual>
+      </link>
+    </xacro:if>
     <!-- Links -->
-    <link name="z_column">
-      <xacro:default_inertial/>
-      <visual>
-        <origin xyz="0 0 0" rpy="0 0 0"/>
-        <geometry>
-          <mesh filename="package://precise_description/meshes/PF3400_Z_Column.STL"/>
-        </geometry>
-        <material name="white"/>
-      </visual>
-    </link>
-    <link name="z_carriage">
-      <xacro:default_inertial/>
-      <visual>
-        <origin xyz="0 0 0" rpy="0 0 0"/>
-        <geometry>
-          <mesh filename="package://precise_description/meshes/PF3400_Z_Carriage.STL"/>
-        </geometry>
-        <material name="white"/>
-      </visual>
-    </link>
-    <link name="inner_link">
-      <xacro:default_inertial/>
-      <visual>
-        <origin xyz="0 0 0" rpy="0 0 0"/>
-        <geometry>
-          <mesh filename="package://precise_description/meshes/PF3400_Inner_Link.STL"/>
-        </geometry>
-        <material name="white"/>
-      </visual>
-    </link>
-    <link name="outer_link">
-      <xacro:default_inertial/>
-      <visual>
-        <origin xyz="0 0 0" rpy="0 0 0"/>
-        <geometry>
-          <mesh filename="package://precise_description/meshes/PF3400_Outer_Link.STL"/>
-        </geometry>
-        <material name="white"/>
-      </visual>
-    </link>
-    <link name="hand">
-      <xacro:default_inertial/>
-      <visual>
-        <origin xyz="0 0 0" rpy="0 0 0"/>
-        <geometry>
-          <mesh filename="package://precise_description/meshes/PF3400_Hand.STL"/>
-        </geometry>
-        <material name="white"/>
-      </visual>
-    </link>
-    <link name="left_finger">
+    <link name="${name}_1_link">
+      <xacro:default_inertial/>
+      <visual>
+        <origin xyz="0 0 0" rpy="0 0 0"/>
+        <geometry>
+          <mesh filename="package://precise_description/meshes/arm_1_link.STL"/>
+        </geometry>
+        <material name="white"/>
+      </visual>
+    </link>
+    <link name="${name}_2_link">
+      <xacro:default_inertial/>
+      <visual>
+        <origin xyz="0 0 0" rpy="0 0 0"/>
+        <geometry>
+          <mesh filename="package://precise_description/meshes/arm_2_link.STL"/>
+        </geometry>
+        <material name="white"/>
+      </visual>
+    </link>
+    <link name="${name}_3_link">
+      <xacro:default_inertial/>
+      <visual>
+        <origin xyz="0 0 0" rpy="0 0 0"/>
+        <geometry>
+          <mesh filename="package://precise_description/meshes/arm_3_link.STL"/>
+        </geometry>
+        <material name="white"/>
+      </visual>
+    </link>
+    <link name="${name}_4_link">
+      <xacro:default_inertial/>
+      <visual>
+        <origin xyz="0 0 0" rpy="0 0 0"/>
+        <geometry>
+          <mesh filename="package://precise_description/meshes/arm_4_link.STL"/>
+        </geometry>
+        <material name="white"/>
+      </visual>
+    </link>
+    <link name="${name}_5_link">
+      <xacro:default_inertial/>
+      <visual>
+        <origin xyz="0 0 0" rpy="0 0 0"/>
+        <geometry>
+          <mesh filename="package://precise_description/meshes/arm_5_link.STL"/>
+        </geometry>
+        <material name="white"/>
+      </visual>
+    </link>
+    <link name="${name}_left_finger">
       <xacro:default_inertial/>
       <visual>
@@ -104,5 +128,5 @@
       </visual>
     </link>
-    <link name="right_finger">
+    <link name="${name}_right_finger">
       <xacro:default_inertial/>
       <visual>
@@ -116,6 +140,6 @@
     <!-- Joints -->
     <joint name="${name}_1_joint" type="prismatic">
-      <parent link="z_column"/>
-      <child link="z_carriage"/>
+      <parent link="${name}_1_link"/>
+      <child link="${name}_2_link"/>
       <axis xyz="0 0 1"/>
       <xacro:insert_block name="origin_1_joint"/>
@@ -123,6 +147,6 @@
     </joint>
     <joint name="${name}_2_joint" type="revolute">
-      <parent link="z_carriage"/>
-      <child link="inner_link"/>
+      <parent link="${name}_2_link"/>
+      <child link="${name}_3_link"/>
       <axis xyz="0 0 1"/>
       <xacro:insert_block name="origin_2_joint"/>
@@ -130,6 +154,6 @@
     </joint>
     <joint name="${name}_3_joint" type="revolute">
-      <parent link="inner_link"/>
-      <child link="outer_link"/>
+      <parent link="${name}_3_link"/>
+      <child link="${name}_4_link"/>
       <axis xyz="0 0 1"/>
       <xacro:insert_block name="origin_3_joint"/>
@@ -137,6 +161,6 @@
     </joint>
     <joint name="${name}_4_joint" type="revolute">
-      <parent link="outer_link"/>
-      <child link="hand"/>
+      <parent link="${name}_4_link"/>
+      <child link="${name}_5_link"/>
       <axis xyz="0 0 1"/>
       <xacro:insert_block name="origin_4_joint"/>
@@ -144,6 +168,6 @@
     </joint>
     <joint name="${name}_5_joint" type="prismatic">
-      <parent link="hand"/>
-      <child link="left_finger"/>
+      <parent link="${name}_5_link"/>
+      <child link="${name}_left_finger"/>
       <axis xyz="0 1 0"/>
       <xacro:insert_block name="origin_5_joint"/>
@@ -151,6 +175,6 @@
     </joint>
     <joint name="${name}_5_mimic_joint" type="prismatic">
-      <parent link="hand"/>
-      <child link="right_finger"/>
+      <parent link="${name}_5_link"/>
+      <child link="${name}_right_finger"/>
       <axis xyz="0 -1 0"/>
       <xacro:insert_block name="origin_5_joint"/>
@@ -161,5 +185,5 @@
     <joint name="gripper_ee_fixed_joint" type="fixed">
       <xacro:insert_block name="origin_gripper_ee_fixed_joint"/>
-      <parent link="hand"/>
+      <parent link="${name}_5_link"/>
       <child link="gripper_ee_fixed_link" />
     </joint>

Commit message: fix xacro.load_yaml deprecation

File: precise_description/robots/PF400_long.urdf.xacro (robot description, xacro)
@@ -3,5 +3,5 @@
        name="PF400_long">
   <xacro:property name="yaml_file" value="$(find precise_description)/robots/PF400_long.yaml"/>
-  <xacro:property name="robot_properties" value="${load_yaml(yaml_file)}"/>
+  <xacro:property name="robot_properties" value="${xacro.load_yaml(yaml_file)}"/>
   <xacro:include filename="$(find precise_description)/urdf/precise_flex.urdf.xacro"/>
   <xacro:precise_flex name="arm" parent="world" has_podest="${True}">

File: precise_description/robots/PF400_short.urdf.xacro (robot description, xacro)
@@ -3,5 +3,5 @@
        name="PF400_short">
   <xacro:property name="yaml_file" value="$(find precise_description)/robots/PF400_short.yaml"/>
-  <xacro:property name="robot_properties" value="${load_yaml(yaml_file)}"/>
+  <xacro:property name="robot_properties" value="${xacro.load_yaml(yaml_file)}"/>
   <xacro:include filename="$(find precise_description)/urdf/precise_flex.urdf.xacro"/>
   <xacro:precise_flex name="arm" parent="world" has_podest="${True}">
