Commit message: harmonize transmission macro

File: precise_description/urdf/common.xacro (robot description, xacro)
@@ -36,13 +36,13 @@
     </inertial>
   </xacro:macro>
-  <xacro:macro name="default_transmission" params="joint_name">
-    <transmission name="${joint_name}_trans">
+  <xacro:macro name="default_transmission" params="jname">
+    <transmission name="${jname}_trans">
       <type>transmission_interface/SimpleTransmission</type>
-      <joint name="${joint_name}">
+      <joint name="${jname}_joint">
         <hardwareInterface>hardware_interface/PositionJointInterface</hardwareInterface>
         <hardwareInterface>hardware_interface/VelocityJointInterface</hardwareInterface>
         <!--hardwareInterface>hardware_interface/EffortJointInterface</hardwareInterface-->
       </joint>
-      <actuator name="${joint_name}_motor">
+      <actuator name="${jname}_motor">
         <mechanicalReduction>1</mechanicalReduction>
       </actuator>

File: precise_description/urdf/transmission.xacro (robot description, xacro)
@@ -3,10 +3,10 @@
   <xacro:include filename="$(find precise_description)/urdf/common.xacro"/>
   <xacro:macro name="precise_flex_transmission" params="name">
-    <xacro:default_transmission joint_name="${name}_1_joint"/>
-    <xacro:default_transmission joint_name="${name}_2_joint"/>
-    <xacro:default_transmission joint_name="${name}_3_joint"/>
-    <xacro:default_transmission joint_name="${name}_4_joint"/>
-    <xacro:default_transmission joint_name="${name}_5_joint"/>
-    <xacro:default_transmission joint_name="${name}_5_mimic_joint"/>
+    <xacro:default_transmission jname="${name}_1_joint"/>
+    <xacro:default_transmission jname="${name}_2_joint"/>
+    <xacro:default_transmission jname="${name}_3_joint"/>
+    <xacro:default_transmission jname="${name}_4_joint"/>
+    <xacro:default_transmission jname="${name}_5_joint"/>
+    <xacro:default_transmission jname="${name}_5_mimic_joint"/>
   </xacro:macro>
 </robot>
