Commit message: rename joints

File: precise_description/urdf/precise_flex.urdf.xacro (robot description, xacro)
@@ -75,5 +75,5 @@
     </link>
     <!-- Joints -->
-    <joint name="Joint1" type="prismatic">
+    <joint name="${name}_1_joint" type="prismatic">
       <parent link="z_column"/>
       <child link="z_carriage"/>
@@ -82,5 +82,5 @@
       <limit effort="1000.0" lower="0.0015" upper="0.4015" velocity="0.5"/>
     </joint>
-    <joint name="Joint2" type="revolute">
+    <joint name="${name}_2_joint" type="revolute">
       <parent link="z_carriage"/>
       <child link="inner_link"/>
@@ -89,5 +89,5 @@
       <limit effort="1000.0" lower="-1.62316" upper="1.62316" velocity="0.5"/>
     </joint>
-    <joint name="Joint3" type="revolute">
+    <joint name="${name}_3_joint" type="revolute">
       <parent link="inner_link"/>
       <child link="outer_link"/>
@@ -96,5 +96,5 @@
       <limit effort="1000.0" lower="0.20944" upper="6.07375" velocity="0.5"/>
     </joint>
-    <joint name="Joint4" type="revolute">
+    <joint name="${name}_4_joint" type="revolute">
       <parent link="outer_link"/>
       <child link="hand"/>
@@ -103,5 +103,5 @@
       <limit effort="1000.0" lower="-16.7552" upper="16.7552" velocity="0.5"/>
     </joint>
-    <joint name="Joint5" type="prismatic">
+    <joint name="${name}_5_joint" type="prismatic">
       <parent link="hand"/>
       <child link="left_finger"/>
@@ -110,5 +110,5 @@
       <limit effort="1000.0" lower="0.051954" upper="0.070" velocity="0.5"/>
     </joint>
-    <joint name="Joint5_mirror" type="prismatic">
+    <joint name="${name}_5_mimic_joint" type="prismatic">
       <parent link="hand"/>
       <child link="right_finger"/>
@@ -116,5 +116,5 @@
       <origin xyz="0.078573 0 -0.04269" rpy="0 0 0"/>
       <limit effort="1000.0" lower="0.051954" upper="0.070" velocity="0.5"/>
-      <mimic joint="Joint5" multiplier="1"/>
+      <mimic joint="${name}_5_joint" multiplier="1"/>
     </joint>
     <!-- extensions -->

File: precise_description/urdf/transmission.xacro (robot description, xacro)
@@ -3,10 +3,10 @@
   <xacro:include filename="$(find precise_description)/urdf/common.xacro"/>
   <xacro:macro name="precise_flex_transmission" params="name">
-    <xacro:default_transmission joint_name="Joint1"/>
-    <xacro:default_transmission joint_name="Joint2"/>
-    <xacro:default_transmission joint_name="Joint3"/>
-    <xacro:default_transmission joint_name="Joint4"/>
-    <xacro:default_transmission joint_name="Joint5"/>
-    <xacro:default_transmission joint_name="Joint5_mirror"/>
+    <xacro:default_transmission joint_name="${name}_1_joint"/>
+    <xacro:default_transmission joint_name="${name}_2_joint"/>
+    <xacro:default_transmission joint_name="${name}_3_joint"/>
+    <xacro:default_transmission joint_name="${name}_4_joint"/>
+    <xacro:default_transmission joint_name="${name}_5_joint"/>
+    <xacro:default_transmission joint_name="${name}_5_mimic_joint"/>
   </xacro:macro>
 </robot>

Commit message: configure joint limits via properties yaml

File: precise_description/urdf/precise_flex.urdf.xacro (robot description, xacro)
@@ -18,4 +18,19 @@
     <xacro:property name="origin_5_joint">
       <origin xyz="${robot_properties['arm']['arm_5_joint']['origin']['x']} ${robot_properties['arm']['arm_5_joint']['origin']['y']} ${robot_properties['arm']['arm_5_joint']['origin']['z']}" rpy="${robot_properties['arm']['arm_5_joint']['origin']['roll']} ${robot_properties['arm']['arm_5_joint']['origin']['pitch']} ${robot_properties['arm']['arm_5_joint']['origin']['yaw']}"/>
+    </xacro:property>
+    <xacro:property name="limit_1_joint">
+      <limit effort="${robot_properties['arm']['arm_1_joint']['limit']['effort']}" lower="${robot_properties['arm']['arm_1_joint']['limit']['lower']}" upper="${robot_properties['arm']['arm_1_joint']['limit']['upper']}" velocity="${robot_properties['arm']['arm_1_joint']['limit']['velocity']}"/>
+    </xacro:property>
+    <xacro:property name="limit_2_joint">
+      <limit effort="${robot_properties['arm']['arm_2_joint']['limit']['effort']}" lower="${robot_properties['arm']['arm_2_joint']['limit']['lower']}" upper="${robot_properties['arm']['arm_2_joint']['limit']['upper']}" velocity="${robot_properties['arm']['arm_2_joint']['limit']['velocity']}"/>
+    </xacro:property>
+    <xacro:property name="limit_3_joint">
+      <limit effort="${robot_properties['arm']['arm_3_joint']['limit']['effort']}" lower="${robot_properties['arm']['arm_3_joint']['limit']['lower']}" upper="${robot_properties['arm']['arm_3_joint']['limit']['upper']}" velocity="${robot_properties['arm']['arm_3_joint']['limit']['velocity']}"/>
+    </xacro:property>
+    <xacro:property name="limit_4_joint">
+      <limit effort="${robot_properties['arm']['arm_4_joint']['limit']['effort']}" lower="${robot_properties['arm']['arm_4_joint']['limit']['lower']}" upper="${robot_properties['arm']['arm_4_joint']['limit']['upper']}" velocity="${robot_properties['arm']['arm_4_joint']['limit']['velocity']}"/>
+    </xacro:property>
+    <xacro:property name="limit_5_joint">
+      <limit effort="${robot_properties['arm']['arm_5_joint']['limit']['effort']}" lower="${robot_properties['arm']['arm_5_joint']['limit']['lower']}" upper="${robot_properties['arm']['arm_5_joint']['limit']['upper']}" velocity="${robot_properties['arm']['arm_5_joint']['limit']['velocity']}"/>
     </xacro:property>
     <!-- mounting -->
@@ -95,5 +110,5 @@
       <axis xyz="0 0 1"/>
       <xacro:insert_block name="origin_1_joint"/>
-      <limit effort="1000.0" lower="0.0015" upper="0.4015" velocity="0.5"/>
+      <xacro:insert_block name="limit_1_joint"/>
     </joint>
     <joint name="${name}_2_joint" type="revolute">
@@ -102,5 +117,5 @@
       <axis xyz="0 0 1"/>
       <xacro:insert_block name="origin_2_joint"/>
-      <limit effort="1000.0" lower="-1.62316" upper="1.62316" velocity="0.5"/>
+      <xacro:insert_block name="limit_2_joint"/>
     </joint>
     <joint name="${name}_3_joint" type="revolute">
@@ -109,5 +124,5 @@
       <axis xyz="0 0 1"/>
       <xacro:insert_block name="origin_3_joint"/>
-      <limit effort="1000.0" lower="0.20944" upper="6.07375" velocity="0.5"/>
+      <xacro:insert_block name="limit_3_joint"/>
     </joint>
     <joint name="${name}_4_joint" type="revolute">
@@ -116,5 +131,5 @@
       <axis xyz="0 0 1"/>
       <xacro:insert_block name="origin_4_joint"/>
-      <limit effort="1000.0" lower="-16.7552" upper="16.7552" velocity="0.5"/>
+      <xacro:insert_block name="limit_4_joint"/>
     </joint>
     <joint name="${name}_5_joint" type="prismatic">
@@ -123,5 +138,5 @@
       <axis xyz="0 1 0"/>
       <xacro:insert_block name="origin_5_joint"/>
-      <limit effort="1000.0" lower="0.051954" upper="0.070" velocity="0.5"/>
+      <xacro:insert_block name="limit_5_joint"/>
     </joint>
     <joint name="${name}_5_mimic_joint" type="prismatic">
@@ -130,5 +145,5 @@
       <axis xyz="0 -1 0"/>
       <xacro:insert_block name="origin_5_joint"/>
-      <limit effort="1000.0" lower="0.051954" upper="0.070" velocity="0.5"/>
+      <xacro:insert_block name="limit_5_joint"/>
       <mimic joint="${name}_5_joint" multiplier="1"/>
     </joint>

Commit message: rescale meshes

File: precise_description/urdf/precise_flex.urdf.xacro (robot description, xacro)
@@ -45,5 +45,5 @@
         <origin xyz="0 0 0" rpy="0 0 0"/>
         <geometry>
-          <mesh filename="package://precise_description/meshes/PF3400_Z_Column.STL" scale="0.001 0.001 0.001"/>
+          <mesh filename="package://precise_description/meshes/PF3400_Z_Column.STL"/>
         </geometry>
         <material name="white"/>
@@ -54,5 +54,5 @@
         <origin xyz="0 0 0" rpy="0 0 0"/>
         <geometry>
-          <mesh filename="package://precise_description/meshes/PF3400_Z_Carriage.STL" scale="0.001 0.001 0.001"/>
+          <mesh filename="package://precise_description/meshes/PF3400_Z_Carriage.STL"/>
         </geometry>
         <material name="white"/>
@@ -63,5 +63,5 @@
         <origin xyz="0 0 0" rpy="0 0 0"/>
         <geometry>
-          <mesh filename="package://precise_description/meshes/PF3400_Inner_Link.STL" scale="0.001 0.001 0.001"/>
+          <mesh filename="package://precise_description/meshes/PF3400_Inner_Link.STL"/>
         </geometry>
         <material name="white"/>
@@ -72,5 +72,5 @@
         <origin xyz="0 0 0" rpy="0 0 0"/>
         <geometry>
-          <mesh filename="package://precise_description/meshes/PF3400_Outer_Link.STL" scale="0.001 0.001 0.001"/>
+          <mesh filename="package://precise_description/meshes/PF3400_Outer_Link.STL"/>
         </geometry>
         <material name="white"/>
@@ -81,5 +81,5 @@
         <origin xyz="0 0 0" rpy="0 0 0"/>
         <geometry>
-          <mesh filename="package://precise_description/meshes/PF3400_Hand.STL" scale="0.001 0.001 0.001"/>
+          <mesh filename="package://precise_description/meshes/PF3400_Hand.STL"/>
         </geometry>
         <material name="white"/>
@@ -90,5 +90,5 @@
         <origin xyz="0 0 0" rpy="0 0 0"/>
         <geometry>
-          <mesh filename="package://precise_description/meshes/PF3400_Left_Finger.STL" scale="0.001 0.001 0.001"/>
+          <mesh filename="package://precise_description/meshes/PF3400_Left_Finger.STL"/>
         </geometry>
         <material name="aluminum"/>
@@ -99,5 +99,5 @@
         <origin xyz="0 0 0" rpy="0 0 0"/>
         <geometry>
-          <mesh filename="package://precise_description/meshes/PF3400_Right_Finger.STL" scale="0.001 0.001 0.001"/>
+          <mesh filename="package://precise_description/meshes/PF3400_Right_Finger.STL"/>
         </geometry>
         <material name="aluminum"/>

Commit message: add gripper_ee_fixed_link

File: precise_description/urdf/precise_flex.urdf.xacro (robot description, xacro)
@@ -155,4 +155,11 @@
       <mimic joint="${name}_5_joint" multiplier="1"/>
     </joint>
+    <!-- endeffector -->
+    <joint name="gripper_ee_fixed_joint" type="fixed">
+      <origin xyz="0 0 0" rpy="0 0 0"/>
+      <parent link="hand"/>
+      <child link="gripper_ee_fixed_link" />
+    </joint>
+    <link name="gripper_ee_fixed_link"/>
     <!-- extensions -->
     <xacro:precise_flex_transmission name="${name}"/>

Commit message: adjust gripper_ee_fixed_link origin

File: precise_description/urdf/precise_flex.urdf.xacro (robot description, xacro)
@@ -157,5 +157,5 @@
     <!-- endeffector -->
     <joint name="gripper_ee_fixed_joint" type="fixed">
-      <origin xyz="0 0 0" rpy="0 0 0"/>
+      <origin xyz="0.0687 0.0 -0.05713" rpy="0 0 0"/>
       <parent link="hand"/>
       <child link="gripper_ee_fixed_link" />

Commit message: gripper_ee_fixed_joint collision free translation

File: precise_description/urdf/precise_flex.urdf.xacro (robot description, xacro)
@@ -157,5 +157,5 @@
     <!-- endeffector -->
     <joint name="gripper_ee_fixed_joint" type="fixed">
-      <origin xyz="0.0687 0.0 -0.05713" rpy="0 0 0"/>
+      <origin xyz="0.0687 0.0 -0.07" rpy="0 0 0" />
       <parent link="hand"/>
       <child link="gripper_ee_fixed_link" />

Commit message: configurable finger meshes

File: precise_description/urdf/precise_flex.urdf.xacro (robot description, xacro)
@@ -96,5 +96,5 @@
         <origin xyz="0 0 0" rpy="0 0 0"/>
         <geometry>
-          <mesh filename="package://precise_description/meshes/PF3400_Left_Finger.STL"/>
+          <mesh filename="${robot_properties['arm']['left_finger']['visual_mesh']}"/>
         </geometry>
         <material name="aluminum"/>
@@ -106,5 +106,5 @@
         <origin xyz="0 0 0" rpy="0 0 0"/>
         <geometry>
-          <mesh filename="package://precise_description/meshes/PF3400_Right_Finger.STL"/>
+          <mesh filename="${robot_properties['arm']['right_finger']['visual_mesh']}"/>
         </geometry>
         <material name="aluminum"/>

Commit message: configurable gripper_ee_fixed_link

File: precise_description/urdf/precise_flex.urdf.xacro (robot description, xacro)
@@ -18,4 +18,7 @@
     <xacro:property name="origin_5_joint">
       <origin xyz="${robot_properties['arm']['arm_5_joint']['origin']['x']} ${robot_properties['arm']['arm_5_joint']['origin']['y']} ${robot_properties['arm']['arm_5_joint']['origin']['z']}" rpy="${robot_properties['arm']['arm_5_joint']['origin']['roll']} ${robot_properties['arm']['arm_5_joint']['origin']['pitch']} ${robot_properties['arm']['arm_5_joint']['origin']['yaw']}"/>
+    </xacro:property>
+    <xacro:property name="origin_gripper_ee_fixed_joint">
+      <origin xyz="${robot_properties['arm']['gripper_ee_fixed_joint']['origin']['x']} ${robot_properties['arm']['gripper_ee_fixed_joint']['origin']['y']} ${robot_properties['arm']['gripper_ee_fixed_joint']['origin']['z']}" rpy="${robot_properties['arm']['gripper_ee_fixed_joint']['origin']['roll']} ${robot_properties['arm']['gripper_ee_fixed_joint']['origin']['pitch']} ${robot_properties['arm']['gripper_ee_fixed_joint']['origin']['yaw']}"/>
     </xacro:property>
     <xacro:property name="limit_1_joint">
@@ -157,5 +160,5 @@
     <!-- endeffector -->
     <joint name="gripper_ee_fixed_joint" type="fixed">
-      <origin xyz="0.0687 0.0 -0.07" rpy="0 0 0" />
+      <xacro:insert_block name="origin_gripper_ee_fixed_joint"/>
       <parent link="hand"/>
       <child link="gripper_ee_fixed_link" />

Commit message: use measurments from kinematic table

File: precise_description/urdf/precise_flex.urdf.xacro (robot description, xacro)
@@ -53,5 +53,5 @@
     <xacro:if value="${has_podest}">
       <joint name="${name}_podest_joint" type="fixed">
-        <origin xyz="0 0 0" rpy="0 0 0"/>
+        <origin xyz="0 0 -0.0096" rpy="0 0 0"/>
         <parent link="${name}_base_link"/>
         <child link="${name}_podest_link"/>
@@ -62,5 +62,5 @@
           <origin xyz="0 0 0" rpy="0 0 0" />
           <geometry>
-            <mesh filename="package://precise_description/meshes/arm_podest_link.STL"/>
+            <mesh filename="${robot_properties['arm']['arm_podest_link']['visual_mesh']}"/>
           </geometry>
         </visual>
@@ -73,5 +73,5 @@
         <origin xyz="0 0 0" rpy="0 0 0"/>
         <geometry>
-          <mesh filename="package://precise_description/meshes/arm_1_link.STL"/>
+          <mesh filename="${robot_properties['arm']['arm_1_link']['visual_mesh']}"/>
         </geometry>
         <material name="white"/>
@@ -83,5 +83,5 @@
         <origin xyz="0 0 0" rpy="0 0 0"/>
         <geometry>
-          <mesh filename="package://precise_description/meshes/arm_2_link.STL"/>
+          <mesh filename="${robot_properties['arm']['arm_2_link']['visual_mesh']}"/>
         </geometry>
         <material name="white"/>
@@ -93,5 +93,5 @@
         <origin xyz="0 0 0" rpy="0 0 0"/>
         <geometry>
-          <mesh filename="package://precise_description/meshes/arm_3_link.STL"/>
+          <mesh filename="${robot_properties['arm']['arm_3_link']['visual_mesh']}"/>
         </geometry>
         <material name="white"/>
@@ -103,5 +103,5 @@
         <origin xyz="0 0 0" rpy="0 0 0"/>
         <geometry>
-          <mesh filename="package://precise_description/meshes/arm_4_link.STL"/>
+          <mesh filename="${robot_properties['arm']['arm_4_link']['visual_mesh']}"/>
         </geometry>
         <material name="white"/>
@@ -113,5 +113,5 @@
         <origin xyz="0 0 0" rpy="0 0 0"/>
         <geometry>
-          <mesh filename="package://precise_description/meshes/arm_5_link.STL"/>
+          <mesh filename="${robot_properties['arm']['arm_5_link']['visual_mesh']}"/>
         </geometry>
         <material name="white"/>

Commit message: fix gazebo_ros_control

File: precise_description/urdf/precise_flex.urdf.xacro (robot description, xacro)
@@ -188,5 +188,7 @@
       <child link="gripper_ee_fixed_link" />
     </joint>
-    <link name="gripper_ee_fixed_link"/>
+    <link name="gripper_ee_fixed_link">
+      <xacro:default_inertial/>
+    </link>
     <!-- extensions -->
     <xacro:precise_flex_transmission name="${name}"/>

File: precise_description/urdf/transmission.xacro (robot description, xacro)
@@ -1,12 +1,12 @@
 <?xml version="1.0"?>
 <robot xmlns:xacro="http://www.ros.org/wiki/xacro">
-  <xacro:include filename="$(find precise_description)/urdf/common.xacro"/>
+  <xacro:include filename="$(find cob_description)/urdf/common.xacro"/>
   <xacro:macro name="precise_flex_transmission" params="name">
-    <xacro:default_transmission jname="${name}_1_joint"/>
-    <xacro:default_transmission jname="${name}_2_joint"/>
-    <xacro:default_transmission jname="${name}_3_joint"/>
-    <xacro:default_transmission jname="${name}_4_joint"/>
-    <xacro:default_transmission jname="${name}_5_joint"/>
-    <xacro:default_transmission jname="${name}_5_mimic_joint"/>
+    <xacro:default_transmission jname="${name}_1"/>
+    <xacro:default_transmission jname="${name}_2"/>
+    <xacro:default_transmission jname="${name}_3"/>
+    <xacro:default_transmission jname="${name}_4"/>
+    <xacro:default_transmission jname="${name}_5"/>
+    <xacro:default_transmission jname="${name}_5_mimic"/>
   </xacro:macro>
 </robot>

Commit message: testing at IPA

File: precise_description/urdf/precise_flex.urdf.xacro (robot description, xacro)
@@ -19,6 +19,12 @@
       <origin xyz="${robot_properties['arm']['arm_5_joint']['origin']['x']} ${robot_properties['arm']['arm_5_joint']['origin']['y']} ${robot_properties['arm']['arm_5_joint']['origin']['z']}" rpy="${robot_properties['arm']['arm_5_joint']['origin']['roll']} ${robot_properties['arm']['arm_5_joint']['origin']['pitch']} ${robot_properties['arm']['arm_5_joint']['origin']['yaw']}"/>
     </xacro:property>
+    <xacro:property name="origin_ee_joint">
+      <origin xyz="${robot_properties['arm']['arm_ee_joint']['origin']['x']} ${robot_properties['arm']['arm_ee_joint']['origin']['y']} ${robot_properties['arm']['arm_ee_joint']['origin']['z']}" rpy="${robot_properties['arm']['arm_ee_joint']['origin']['roll']} ${robot_properties['arm']['arm_ee_joint']['origin']['pitch']} ${robot_properties['arm']['arm_ee_joint']['origin']['yaw']}"/>
+    </xacro:property>
     <xacro:property name="origin_gripper_ee_fixed_joint">
       <origin xyz="${robot_properties['arm']['gripper_ee_fixed_joint']['origin']['x']} ${robot_properties['arm']['gripper_ee_fixed_joint']['origin']['y']} ${robot_properties['arm']['gripper_ee_fixed_joint']['origin']['z']}" rpy="${robot_properties['arm']['gripper_ee_fixed_joint']['origin']['roll']} ${robot_properties['arm']['gripper_ee_fixed_joint']['origin']['pitch']} ${robot_properties['arm']['gripper_ee_fixed_joint']['origin']['yaw']}"/>
+    </xacro:property>
+    <xacro:property name="origin_gripper_ee_joint">
+      <origin xyz="${robot_properties['arm']['gripper_ee_joint']['origin']['x']} ${robot_properties['arm']['gripper_ee_joint']['origin']['y']} ${robot_properties['arm']['gripper_ee_joint']['origin']['z']}" rpy="${robot_properties['arm']['gripper_ee_joint']['origin']['roll']} ${robot_properties['arm']['gripper_ee_joint']['origin']['pitch']} ${robot_properties['arm']['gripper_ee_joint']['origin']['yaw']}"/>
     </xacro:property>
     <xacro:property name="limit_1_joint">
@@ -65,4 +71,10 @@
           </geometry>
         </visual>
+        <collision>
+          <origin xyz="0 0 0" rpy="0 0 0" />
+          <geometry>
+            <mesh filename="${robot_properties['arm']['arm_podest_link']['visual_mesh']}"/>
+          </geometry>
+        </collision>
       </link>
     </xacro:if>
@@ -77,4 +89,11 @@
         <material name="white"/>
       </visual>
+      <collision>
+        <origin xyz="0 0 0" rpy="0 0 0"/>
+        <geometry>
+          <mesh filename="${robot_properties['arm']['arm_1_link']['visual_mesh']}"/>
+        </geometry>
+        <material name="white"/>
+      </collision>
     </link>
     <link name="${name}_2_link">
@@ -87,4 +106,11 @@
         <material name="white"/>
       </visual>
+      <collision>
+        <origin xyz="0 0 0" rpy="0 0 0"/>
+        <geometry>
+          <mesh filename="${robot_properties['arm']['arm_2_link']['visual_mesh']}"/>
+        </geometry>
+        <material name="white"/>
+      </collision>
     </link>
     <link name="${name}_3_link">
@@ -97,4 +123,11 @@
         <material name="white"/>
       </visual>
+      <collision>
+        <origin xyz="0 0 0" rpy="0 0 0"/>
+        <geometry>
+          <mesh filename="${robot_properties['arm']['arm_3_link']['visual_mesh']}"/>
+        </geometry>
+        <material name="white"/>
+      </collision>
     </link>
     <link name="${name}_4_link">
@@ -107,4 +140,11 @@
         <material name="white"/>
       </visual>
+      <collision>
+        <origin xyz="0 0 0" rpy="0 0 0"/>
+        <geometry>
+          <mesh filename="${robot_properties['arm']['arm_4_link']['visual_mesh']}"/>
+        </geometry>
+        <material name="white"/>
+      </collision>
     </link>
     <link name="${name}_5_link">
@@ -117,4 +157,11 @@
         <material name="white"/>
       </visual>
+      <collision>
+        <origin xyz="0 0 0" rpy="0 0 0"/>
+        <geometry>
+          <mesh filename="${robot_properties['arm']['arm_5_link']['visual_mesh']}"/>
+        </geometry>
+        <material name="white"/>
+      </collision>
     </link>
     <link name="${name}_left_finger">
@@ -127,4 +174,11 @@
         <material name="aluminum"/>
       </visual>
+      <collision>
+        <origin xyz="0 0 0" rpy="0 0 0"/>
+        <geometry>
+          <mesh filename="${robot_properties['arm']['left_finger']['visual_mesh']}"/>
+        </geometry>
+        <material name="aluminum"/>
+      </collision>
     </link>
     <link name="${name}_right_finger">
@@ -137,4 +191,11 @@
         <material name="aluminum"/>
       </visual>
+      <collision>
+        <origin xyz="0 0 0" rpy="0 0 0"/>
+        <geometry>
+          <mesh filename="${robot_properties['arm']['right_finger']['visual_mesh']}"/>
+        </geometry>
+        <material name="aluminum"/>
+      </collision>
     </link>
     <!-- Joints -->
@@ -183,10 +244,26 @@
     </joint>
     <!-- endeffector -->
+    <joint name="${name}_ee_joint" type="fixed">
+      <xacro:insert_block name="origin_ee_joint"/>
+      <parent link="${name}_5_link"/>
+      <child link="${name}_ee_link" />
+    </joint>
+    <link name="${name}_ee_link">
+      <xacro:default_inertial/>
+    </link>
     <joint name="gripper_ee_fixed_joint" type="fixed">
       <xacro:insert_block name="origin_gripper_ee_fixed_joint"/>
-      <parent link="${name}_5_link"/>
+      <parent link="${name}_ee_link"/>
       <child link="gripper_ee_fixed_link" />
     </joint>
     <link name="gripper_ee_fixed_link">
+      <xacro:default_inertial/>
+    </link>
+    <joint name="gripper_ee_joint" type="fixed">
+      <xacro:insert_block name="origin_gripper_ee_joint"/>
+      <parent link="${name}_ee_link"/>
+      <child link="gripper_ee_link" />
+    </joint>
+    <link name="gripper_ee_link">
       <xacro:default_inertial/>
     </link>
