Commit message: move gripper description to external xacro

File: precise_description/urdf/precise_flex.urdf.xacro (robot description, xacro)
@@ -165,37 +165,9 @@
       </collision>
     </link>
-    <link name="${name}_left_finger">
-      <xacro:default_inertial/>
-      <visual>
-        <origin xyz="0 0 0" rpy="0 0 0"/>
-        <geometry>
-          <mesh filename="${robot_properties['arm']['left_finger']['visual_mesh']}"/>
-        </geometry>
-        <material name="aluminum"/>
-      </visual>
-      <collision>
-        <origin xyz="0 0 0" rpy="0 0 0"/>
-        <geometry>
-          <mesh filename="${robot_properties['arm']['left_finger']['visual_mesh']}"/>
-        </geometry>
-        <material name="aluminum"/>
-      </collision>
-    </link>
-    <link name="${name}_right_finger">
-      <xacro:default_inertial/>
-      <visual>
-        <origin xyz="0 0 0" rpy="0 0 0"/>
-        <geometry>
-          <mesh filename="${robot_properties['arm']['right_finger']['visual_mesh']}"/>
-        </geometry>
-        <material name="aluminum"/>
-      </visual>
-      <collision>
-        <origin xyz="0 0 0" rpy="0 0 0"/>
-        <geometry>
-          <mesh filename="${robot_properties['arm']['right_finger']['visual_mesh']}"/>
-        </geometry>
-        <material name="aluminum"/>
-      </collision>
+    <link name="${name}_left_finger_mount_link">
+      <xacro:default_inertial/>
+    </link>
+    <link name="${name}_right_finger_mount_link">
+      <xacro:default_inertial/>
     </link>
     <!-- Joints -->
@@ -230,5 +202,5 @@
     <joint name="${name}_5_joint" type="prismatic">
       <parent link="${name}_5_link"/>
-      <child link="${name}_left_finger"/>
+      <child link="${name}_left_finger_mount_link"/>
       <axis xyz="0 1 0"/>
       <xacro:insert_block name="origin_5_joint"/>
@@ -237,5 +209,5 @@
     <joint name="${name}_5_mimic_joint" type="prismatic">
       <parent link="${name}_5_link"/>
-      <child link="${name}_right_finger"/>
+      <child link="${name}_right_finger_mount_link"/>
       <axis xyz="0 -1 0"/>
       <xacro:insert_block name="origin_5_joint"/>
@@ -250,20 +222,4 @@
     </joint>
     <link name="${name}_ee_link">
-      <xacro:default_inertial/>
-    </link>
-    <joint name="gripper_ee_fixed_joint" type="fixed">
-      <xacro:insert_block name="origin_gripper_ee_fixed_joint"/>
-      <parent link="${name}_ee_link"/>
-      <child link="gripper_ee_fixed_link" />
-    </joint>
-    <link name="gripper_ee_fixed_link">
-      <xacro:default_inertial/>
-    </link>
-    <joint name="gripper_ee_joint" type="fixed">
-      <xacro:insert_block name="origin_gripper_ee_joint"/>
-      <parent link="${name}_ee_link"/>
-      <child link="gripper_ee_link" />
-    </joint>
-    <link name="gripper_ee_link">
       <xacro:default_inertial/>
     </link>
