Commit message: explicit material definition

File: precise_description/urdf/gripper.urdf.xacro (robot description, xacro)
@@ -2,4 +2,7 @@
 <robot xmlns:xacro="http://www.ros.org/wiki/xacro">
   <xacro:macro name="gripper" params="name parent parent_left_finger parent_right_finger *origin *origin_left_finger *origin_right_finger">
+    <material name="precise_aluminum">
+      <color rgba="0.6 0.6 0.6 1"/>
+    </material>
     <joint name="${name}_ee_fixed_joint" type="fixed">
       <xacro:insert_block name="origin"/>
@@ -30,5 +33,5 @@
           <mesh filename="package://precise_description/meshes/mrk_finger.STL"/>
         </geometry>
-        <material name="aluminum"/>
+        <material name="precise_aluminum"/>
       </visual>
       <collision>
@@ -37,5 +40,5 @@
           <mesh filename="package://precise_description/meshes/mrk_finger.STL"/>
         </geometry>
-        <material name="aluminum"/>
+        <material name="precise_aluminum"/>
       </collision>
     </link>
@@ -52,5 +55,5 @@
           <mesh filename="package://precise_description/meshes/mrk_finger.STL"/>
         </geometry>
-        <material name="aluminum"/>
+        <material name="precise_aluminum"/>
       </visual>
       <collision>
@@ -59,5 +62,5 @@
           <mesh filename="package://precise_description/meshes/mrk_finger.STL"/>
         </geometry>
-        <material name="aluminum"/>
+        <material name="precise_aluminum"/>
       </collision>
     </link>

File: precise_description/urdf/precise_flex.urdf.xacro (robot description, xacro)
@@ -1,5 +1,4 @@
 <?xml version="1.0"?>
 <robot xmlns:xacro="http://www.ros.org/wiki/xacro">
-  <xacro:include filename="$(find precise_description)/urdf/materials.xacro"/>
   <xacro:include filename="$(find precise_description)/urdf/transmission.xacro" />
   <xacro:macro name="precise_flex" params="parent name *origin has_podest:=True">
@@ -43,4 +42,7 @@
       <limit effort="${robot_properties['arm']['arm_5_joint']['limit']['effort']}" lower="${robot_properties['arm']['arm_5_joint']['limit']['lower']}" upper="${robot_properties['arm']['arm_5_joint']['limit']['upper']}" velocity="${robot_properties['arm']['arm_5_joint']['limit']['velocity']}"/>
     </xacro:property>
+    <material name="precise_white">
+      <color rgba="1 1 1 1"/>
+    </material>
     <!-- mounting -->
     <joint name="${name}_base_joint" type="fixed">
@@ -87,5 +89,5 @@
           <mesh filename="${robot_properties['arm']['arm_1_link']['visual_mesh']}"/>
         </geometry>
-        <material name="white"/>
+        <material name="precise_white"/>
       </visual>
       <collision>
@@ -94,5 +96,5 @@
           <mesh filename="${robot_properties['arm']['arm_1_link']['visual_mesh']}"/>
         </geometry>
-        <material name="white"/>
+        <material name="precise_white"/>
       </collision>
     </link>
@@ -104,5 +106,5 @@
           <mesh filename="${robot_properties['arm']['arm_2_link']['visual_mesh']}"/>
         </geometry>
-        <material name="white"/>
+        <material name="precise_white"/>
       </visual>
       <collision>
@@ -111,5 +113,5 @@
           <mesh filename="${robot_properties['arm']['arm_2_link']['visual_mesh']}"/>
         </geometry>
-        <material name="white"/>
+        <material name="precise_white"/>
       </collision>
     </link>
@@ -121,5 +123,5 @@
           <mesh filename="${robot_properties['arm']['arm_3_link']['visual_mesh']}"/>
         </geometry>
-        <material name="white"/>
+        <material name="precise_white"/>
       </visual>
       <collision>
@@ -128,5 +130,5 @@
           <mesh filename="${robot_properties['arm']['arm_3_link']['visual_mesh']}"/>
         </geometry>
-        <material name="white"/>
+        <material name="precise_white"/>
       </collision>
     </link>
@@ -138,5 +140,5 @@
           <mesh filename="${robot_properties['arm']['arm_4_link']['visual_mesh']}"/>
         </geometry>
-        <material name="white"/>
+        <material name="precise_white"/>
       </visual>
       <collision>
@@ -145,5 +147,5 @@
           <mesh filename="${robot_properties['arm']['arm_4_link']['visual_mesh']}"/>
         </geometry>
-        <material name="white"/>
+        <material name="precise_white"/>
       </collision>
     </link>
@@ -155,5 +157,5 @@
           <mesh filename="${robot_properties['arm']['arm_5_link']['visual_mesh']}"/>
         </geometry>
-        <material name="white"/>
+        <material name="precise_white"/>
       </visual>
       <collision>
@@ -162,5 +164,5 @@
           <mesh filename="${robot_properties['arm']['arm_5_link']['visual_mesh']}"/>
         </geometry>
-        <material name="white"/>
+        <material name="precise_white"/>
       </collision>
     </link>

Commit message: longer collision mesh for finger

File: precise_description/urdf/gripper.urdf.xacro (robot description, xacro)
@@ -38,5 +38,5 @@
         <origin xyz="0 0 0" rpy="0 0 0"/>
         <geometry>
-          <mesh filename="package://precise_description/meshes/mrk_finger.STL"/>
+          <mesh filename="package://precise_description/meshes/mrk_finger_collision.STL"/>
         </geometry>
         <material name="precise_aluminum"/>
@@ -60,5 +60,5 @@
         <origin xyz="0 0 0" rpy="0 0 0"/>
         <geometry>
-          <mesh filename="package://precise_description/meshes/mrk_finger.STL"/>
+          <mesh filename="package://precise_description/meshes/mrk_finger_collision.STL"/>
         </geometry>
         <material name="precise_aluminum"/>
